File: antispark-pcb/antispark-pcb.kicad_pcb (KiCad board)
At the start: 2 copper layers, 50 x 40 mm, 15 parts, among them P1 PAD_SOLDER_5mm, P2 PAD_SOLDER_5mm, P3 JST_GH_6_RA, P4 PAD_SOLDER_5mm, P5 PAD_SOLDER_5mm, Q1 IRF7749L2, Q2 IRF7749L2, Q3 IRF7749L2, Q4 IRF7749L2, Q5 IRF7749L2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

Commit message: Minor tidy and positioning of text
Cleanup of pours and text locations for cleaner appearance.
Routing:
- net GNDPWR: track 0.00 -> 18.5 mm, vias 34 -> 36
- net Net-(P3-Pad6): track 1.83 -> 0.00 mm, vias 1 -> 0
- net Net-(P3-Pad5): track 1.83 -> 0.00 mm, vias 1 -> 0
- net GATE: track 91.5 -> 92.7 mm
Changed lines of the file:
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@@
     (thickness 1.6)
     (drawings 17)
-    (tracks 173)
+    (tracks 178)
     (zones 0)
     (modules 15)
@@
     (pad_to_paste_clearance_ratio -0.08)
     (aux_axis_origin 100 100)
-    (grid_origin 100 100)
     (visible_elements FFFDFF7F)
     (pcbplotparams
@@
   )
   (module Applidyne_Special:directFET_L8 (layer F.Cu)
-    (at 119.4 115 90)
+    (at 119.39964 114.99912 90)
     (descr "IR-directFET, L8-Outline, Pads with Names,")
     (tags "IR-directFET, L8-Outline, Pads with Names,")
@@
     (effects (font (size 1.5 1.5) (thickness 0.3)) (justify mirror))
   )
-  (gr_text LOAD (at 146 121 90) (layer B.SilkS)
+  (gr_text LOAD (at 147.3 121 90) (layer B.SilkS)
     (effects (font (size 1.5 1.5) (thickness 0.3)) (justify mirror))
   )
@@
     (effects (font (size 1 1) (thickness 0.15)))
   )
-  (gr_text BATTERY (at 112.2 121 90) (layer F.Mask)
+  (gr_text BATTERY (at 110 120.8 90) (layer F.Mask)
     (effects (font (size 1.5 1.5) (thickness 0.3)))
   )
-  (gr_text LOAD (at 146 121 90) (layer F.Mask)
+  (gr_text LOAD (at 147.3 121 90) (layer F.Mask)
     (effects (font (size 1.5 1.5) (thickness 0.3)))
   )
@@
   (gr_line (start 100 100) (end 100 140) (layer Edge.Cuts) (width 0.15))
   (gr_line (start 100 100) (end 150 100) (layer Edge.Cuts) (width 0.15))
+  (segment (start 103 124.4) (end 103 123.7) (width 0.35) (layer B.Cu) (net 1))
+  (segment (start 103 123.7) (end 106.3 120.4) (width 0.35) (layer B.Cu) (net 1))
+  (segment (start 106.3 120.4) (end 113.5 120.4) (width 0.35) (layer B.Cu) (net 1))
+  (segment (start 113.5 120.4) (end 114.600001 119.299999) (width 0.35) (layer B.Cu) (net 1))
+  (segment (start 114.600001 119.299999) (end 115 118.9) (width 0.35) (layer B.Cu) (net 1))
+  (segment (start 101.6 124.4) (end 103 124.4) (width 0.35) (layer F.Cu) (net 1))
+  (via (at 103 124.4) (size 0.8) (drill 0.4) (layers F.Cu B.Cu) (net 1))
+  (segment (start 117.2 119.5) (end 115.6 119.5) (width 0.4) (layer F.Cu) (net 1))
+  (segment (start 115.6 119.5) (end 115 118.9) (width 0.4) (layer F.Cu) (net 1))
+  (via (at 115 118.9) (size 0.8) (drill 0.4) (layers F.Cu B.Cu) (net 1))
   (via (at 133.2 121) (size 0.8) (drill 0.4) (layers F.Cu B.Cu) (net 1))
   (via (at 137.6 123) (size 0.8) (drill 0.4) (layers F.Cu B.Cu) (net 1))
@@
   (segment (start 105 125.2) (end 105 124.85) (width 0.3) (layer F.Cu) (net 2))
   (segment (start 105 124.85) (end 104.55 124.4) (width 0.3) (layer F.Cu) (net 2))
+  (segment (start 117.6 126.5) (end 117.6 125.5) (width 0.6) (layer B.Cu) (net 3))
+  (segment (start 117.6 125.5) (end 114.5 122.4) (width 0.6) (layer B.Cu) (net 3))
+  (segment (start 114.5 122.4) (end 107 122.4) (width 0.6) (layer B.Cu) (net 3))
+  (segment (start 107 122.4) (end 106.6 122) (width 0.6) (layer B.Cu) (net 3))
+  (segment (start 117.6 117.4) (end 117.6 118.5) (width 0.6) (layer B.Cu) (net 3))
+  (segment (start 117.6 118.5) (end 114.7 121.4) (width 0.6) (layer B.Cu) (net 3))
+  (segment (start 114.7 121.4) (end 107 121.4) (width 0.6) (layer B.Cu) (net 3))
+  (segment (start 107 121.4) (end 106.6 121.8) (width 0.6) (layer B.Cu) (net 3))
   (segment (start 106.6 121.8) (end 104.8 121.8) (width 0.25) (layer F.Cu) (net 3))
   (segment (start 104.8 121.8) (end 103.2 120.2) (width 0.25) (layer F.Cu) (net 3))
@@
   (segment (start 104.4 124) (end 106.6 121.8) (width 0.4) (layer B.Cu) (net 3))
   (segment (start 117.6 126.6) (end 117.6 126.5) (width 0.25) (layer B.Cu) (net 3))
-  (segment (start 117.6 126.5) (end 113.5 122.4) (width 0.6) (layer B.Cu) (net 3))
-  (segment (start 113.5 122.4) (end 107 122.4) (width 0.6) (layer B.Cu) (net 3))
-  (segment (start 107 122.4) (end 106.6 122) (width 0.6) (layer B.Cu) (net 3))
   (segment (start 106.6 122) (end 106.6 121.8) (width 0.25) (layer B.Cu) (net 3))
-  (segment (start 107.3 121.4) (end 107 121.4) (width 0.6) (layer B.Cu) (net 3))
-  (segment (start 107 121.4) (end 106.6 121.8) (width 0.6) (layer B.Cu) (net 3))
   (via (at 106.6 121.8) (size 0.8) (drill 0.4) (layers F.Cu B.Cu) (net 3))
-  (segment (start 113.6 121.4) (end 107.3 121.4) (width 0.6) (layer B.Cu) (net 3))
-  (segment (start 117.6 117.4) (end 113.6 121.4) (width 0.6) (layer B.Cu) (net 3))
   (segment (start 125.6 126.6) (end 125.034315 126.6) (width 0.6) (layer B.Cu) (net 3))
   (segment (start 125.034315 126.6) (end 117.6 126.6) (width 0.6) (layer B.Cu) (net 3))
@@
   (segment (start 117.74956 117.25044) (end 117.6 117.4) (width 0.5) (layer F.Cu) (net 3))
   (via (at 117.6 117.4) (size 0.8) (drill 0.4) (layers F.Cu B.Cu) (net 3))
-  (segment (start 105 119.725) (end 106.725 119.725) (width 0.25) (layer F.Cu) (net 9))
-  (segment (start 106.725 119.725) (end 106.8 119.8) (width 0.25) (layer F.Cu) (net 9))
-  (via (at 106.8 119.8) (size 0.8) (drill 0.4) (layers F.Cu B.Cu) (net 9))
   (segment (start 103.425 109.8) (end 103.425 107.025) (width 0.25) (layer F.Cu) (net 4))
   (segment (start 103.425 107.025) (end 103.4 107) (width 0.25) (layer F.Cu) (net 4))
@@
   (segment (start 104.975 113.45) (end 105 113.475) (width 0.25) (layer F.Cu) (net 5))
   (segment (start 104.975 113.65) (end 105 113.675) (width 0.25) (layer F.Cu) (net 5))
-  (segment (start 105 118.475) (end 106.725 118.475) (width 0.25) (layer F.Cu) (net 8))
-  (segment (start 106.725 118.475) (end 106.8 118.4) (width 0.25) (layer F.Cu) (net 8))
-  (via (at 106.8 118.4) (size 0.8) (drill 0.4) (layers F.Cu B.Cu) (net 8))
   (via (at 137.1 114.4) (size 0.8) (drill 0.4) (layers F.Cu B.Cu) (net 7))
   (via (at 136 114.4) (size 0.8) (drill 0.4) (layers F.Cu B.Cu) (net 7))
@@
       (pts
         (xy 150 140) (xy 115.8 140) (xy 115.8 132.2) (xy 139 132.2) (xy 139 125.8)
-        (xy 115.8 125.8) (xy 115.8 118.2) (xy 139 118.2) (xy 139 111.8) (xy 115.8 111.8)
-        (xy 115.8 108.4) (xy 150 108.4)
+        (xy 117.6 125.8) (xy 115.8 123.9) (xy 115.8 118.2) (xy 139 118.2) (xy 139 111.8)
+        (xy 115.8 111.8) (xy 115.8 108.4) (xy 150 108.4)
       )
     )
@@
         (xy 138.8 126) (xy 138.8 132) (xy 115.6 132) (xy 115.6 140) (xy 100 140)
         (xy 100 130.8) (xy 107.8 130.8) (xy 107.8 108.4) (xy 115.6 108.4) (xy 115.6 112)
-        (xy 138.8 112) (xy 138.8 118) (xy 115.6 118) (xy 115.6 126)
+        (xy 138.8 112) (xy 138.8 118) (xy 115.6 118) (xy 115.6 123.5) (xy 118.1 126)
       )
     )
